File: BQ24650_1U_SolarChargerBoard copy.kicad_pcb (KiCad board)
At the start: 2 copper layers, 48 parts, among them J1 CE_MPPSET, J2 solar+, J3 solar-, J4 BATT+, J5 BATT-, J6 TS, Q1 Q_NMOS_GDS, Q2 Q_NMOS_GDS, Q3 Q_NMOS_GDS, U1 BQ24650

Commit message: placing and trace
Parts:
- Q1, Q2, R12: moved to B.Cu
- moved R12 103.8 mm to (126.7, 81.6), turned to -90 degrees
- moved Q2 98.3 mm to (129.2, 88.8), turned to 180 degrees
- moved Q1 91.4 mm to (136.3, 90.5), turned to -90 degrees
- moved R5 80.2 mm to (148.1, 91.7), turned to 90 degrees
- moved D2 79.5 mm to (126.2, 86.5), turned to 180 degrees
- moved TP4 78.5 mm to (122.8, 78.5)
- moved TP6 78.5 mm to (122.7, 84.8)
- moved TP2 77.7 mm to (122.7, 90.8)
- moved C9 73.4 mm to (126.0, 80.5), turned to 180 degrees
- moved L1 73.2 mm to (129.7, 93.2), turned to 180 degrees
- moved C8 71.7 mm to (126.0, 82.8), turned to 180 degrees
- moved TP5 71.0 mm to (135.6, 95.5)
- moved C7 68.2 mm to (129.1, 81.5), turned to 90 degrees
- moved TP1 66.6 mm to (139.0, 95.5)
- moved TP9 65.4 mm to (137.9, 75.2)
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Routing:
- net Vin: track 0.00 -> 29.7 mm, vias 0 -> 2
- net MPPSET: track 0.00 -> 23.8 mm
- net PH: track 0.00 -> 21.2 mm, vias 0 -> 2
- net SRP: track 0.00 -> 19.3 mm, vias 0 -> 2
- net SRN: track 0.00 -> 18.9 mm, vias 0 -> 1
- net /Vin-D1: track 0.00 -> 17.4 mm, vias 0 -> 1
- net VFB: track 0.00 -> 16.2 mm
- net BTST: track 0.00 -> 13.8 mm
- net VCC: track 0.00 -> 13.1 mm
- net REGN: track 0.00 -> 12.5 mm
- net TS: track 0.00 -> 11.6 mm, vias 0 -> 2
- net VREF: track 0.00 -> 10.9 mm
- net Net-(R1-Pad1): track 0.00 -> 6.57 mm
- net Net-(R4-Pad2): track 0.00 -> 6.42 mm
- net Net-(C1-Pad1): track 0.00 -> 4.58 mm
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- added copper zone on B.Cu, net GND
- added copper zone on F.Cu, net GND
Other:
- board outline added: 33 x 23 mm
