File: BQ24650_1U_SolarChargerBoard copy.kicad_pcb (KiCad board)
At the start: 2 copper layers, 48 parts, among them J1 CE_MPPSET, J2 solar+, J3 solar-, J4 BATT+, J5 BATT-, J6 TS, Q1 Q_NMOS_GDS, Q2 Q_NMOS_GDS, Q3 Q_NMOS_GDS, U1 BQ24650

Commit message: new layout
Parts:
- R1, R10, R11, R2, R3, R4, R7, R8, R9: footprint Resistor_SMD:R_0402_1005Metric -> Resistor_SMD:R_0603_1608Metric_Pad0.98x0.95mm_HandSolder
- R5: footprint Resistor_SMD:R_2512_6332Metric -> Resistor_SMD:R_0805_2012Metric
- TP1, TP2, TP3, TP4, TP5, TP6, TP7, TP8, TP9: moved to B.Cu
- moved R5 107.5 mm to (122.6, 78.5), turned to 90 degrees
- moved Q1 91.7 mm to (135.9, 77.6), turned to 90 degrees
- moved Q2 86.9 mm to (141.5, 77.6), turned to 90 degrees
- moved R12 85.3 mm to (146.9, 78.0), turned to -90 degrees
- moved TP8 80.4 mm to (126.5, 89.4), turned to 180 degrees
- moved Q3 80.1 mm to (126.6, 86.5)
- moved TP7 76.9 mm to (134.3, 95.6), turned to 180 degrees
- moved TP3 74.9 mm to (124.0, 89.3), turned to 180 degrees
- moved R6 69.9 mm to (126.7, 75.1), turned to 180 degrees
- moved TP4 69.2 mm to (139.5, 95.5), turned to 180 degrees
- moved TP1 68.5 mm to (128.9, 75.4), turned to 180 degrees
- moved C6 66.6 mm to (130.1, 77.5), turned to 180 degrees
- moved D4 66.4 mm to (129.3, 83.4), turned to 90 degrees
- moved D2 66.3 mm to (140.4, 83.5), turned to 90 degrees
- moved RV2 66.3 mm to (124.0, 91.1), turned to 180 degrees
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Other:
- board outline added: 33 x 23 mm
- board text removed: "Front board"
- board text removed: "Hole"
- board text removed: "can be on the Back side, if there is less space"
- board text removed: "things to be on the edge or accessible"

Commit message: layout done
Parts:
- R1, R2, R3, R4: footprint Resistor_SMD:R_0603_1608Metric_Pad0.98x0.95mm_HandSolder -> Resistor_SMD:R_0805_2012Metric_Pad1.20x1.40mm_HandSolder
- moved R2 15.4 mm to (138.7, 93.5), turned to 180 degrees
- moved R4 9.63 mm to (134.5, 95.5), turned to 180 degrees
- moved R3 8.68 mm to (134.5, 93.5), turned to 180 degrees
- moved R9 5.84 mm to (132.6, 89.2), turned to -90 degrees
- moved TP7 5.47 mm to (132.9, 90.3)
- moved TP4 5.12 mm to (143.6, 92.3)
- moved RV2 5.11 mm to (129.1, 91.0), turned to 0 degrees
- moved TP3 4.70 mm to (128.6, 88.5)
- moved R1 3.29 mm to (138.7, 95.5), turned to 180 degrees
- moved R11 2.68 mm to (138.6, 91.6), turned to 180 degrees
- moved C10 1.67 mm to (151.5, 85.8), turned to -90 degrees
- moved Q3 1.63 mm to (128.2, 86.5)
- moved R10 1.59 mm to (130.3, 94.6)
- moved C3 1.37 mm to (135.1, 91.3), turned to 0 degrees
- moved TP8 1.02 mm to (126.0, 88.4)
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Routing:
- net SRN: track 0.00 -> 44.5 mm, vias 0 -> 2
- net Vin: track 0.00 -> 32.4 mm
- net VFB: track 0.00 -> 28.4 mm
- net SRP: track 0.00 -> 24.9 mm
- net MPPSET: track 0.00 -> 22.3 mm, vias 0 -> 3
- net /Vin-D1: track 0.00 -> 17.7 mm, vias 0 -> 2
- net PH: track 0.00 -> 17.0 mm, vias 0 -> 3
- net VCC: track 0.00 -> 15.1 mm, vias 0 -> 1
- net TS: track 0.00 -> 13.5 mm, vias 0 -> 2
- net STAT2: track 0.00 -> 10.0 mm
- net Net-(R4-Pad2): track 0.00 -> 9.62 mm, vias 0 -> 1
- net Net-(R1-Pad1): track 0.00 -> 7.12 mm, vias 0 -> 1
- net BTST: track 0.00 -> 7.07 mm, vias 0 -> 2
- net VREF: track 0.00 -> 6.91 mm, vias 0 -> 1
- net GND: track 0.00 -> 6.46 mm, vias 0 -> 27
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- added copper zone on B.Cu, net GND
- added copper zone on F.Cu, net GND
Other:
- board text added: "-"
- board text added: "BATT+"
- board text added: "CE"
- board text added: "TS"
- board text added: "VIN+"
